File: SolarCanLantern.sch (KiCad schematic (older format))
At the start: 19 parts, among them IC1 ATTINY13A-SS, J2-1 Solar_Cell, Q1 MMBT2222L_NPN_NG, Q2 MMBT2222L_NPN_NG, Q3 MMBT2222L_NPN_NG, Q4 NX700_NMOS_NG

Commit message: resolved some library problems and switched to mosfets as a test
Parts:
- removed D2: BAT54_SCHOTTKY_NG, symbol BAT54_SCHOTTKY_NG
- removed D4: LED, symbol LED
- removed IC1: ATTINY13A-SS, symbol ATTINY13A-SS
- removed J2-1: Solar_Cell, symbol Solar_Cell
- removed Q1, Q2, Q3: MMBT2222L_NPN_NG, symbol MMBT2222L_NPN_NG
- removed Q4: NX700_NMOS_NG, symbol NX700_NMOS_NG
- removed R6: 1k, symbol R
- removed R8, R9: 10, symbol R
- removed S1: SHURTERPBSW_NG, symbol SHURTERPBSW_NG
- added BT1: Battery_Cell, symbol Battery_Cell
- added D2: LED, LEDs:LED_0805_HandSoldering, symbol LED
- added D4: D, Diodes_SMD:D_0805, symbol D
- added Q1, Q2, Q3, Q4: 2N7002, TO_SOT_Packages_SMD:SOT-23, symbol 2N7002
- added SC1: Solar_Cell, symbol Solar_Cell
- added U1: ATTINY13-20SSU, Housings_SOIC:SOIC-8_3.9x4.9mm_Pitch1.27mm, symbol ATTINY13-20SSU
- D1, D3: footprint (none) -> LEDs:LED_0805_HandSoldering
- R1: value 1k -> 287K; footprint (none) -> Resistors_SMD:R_0805_HandSoldering
- R2: value 10 -> 88.7K; footprint (none) -> Resistors_SMD:R_0805_HandSoldering
- R3: value 88.7k -> 10Ω; footprint (none) -> Resistors_SMD:R_0805_HandSoldering
- R4: value 287k -> 10Ω; footprint (none) -> Resistors_SMD:R_0805_HandSoldering
- R5: value 1k -> 10Ω; footprint (none) -> Resistors_SMD:R_0805_HandSoldering
Connections:
- net labels added: LEDA, LEDB, LEDC, Switch, VBatt_Divider, ~SOLAR
- wire segments 32 -> 33
Other:
- note added: "Note: There are only 2 PWM capable pins so\nLEDS A and B are on PWM capable pins, while C is not"
- note added: "switch\n"
